File: pwrcon_1.sch (KiCad schematic (older format))
At the start: 53 parts, among them J1 CON3, J4 CON3, J5 Conn_01x03_Female, J6 Conn_01x04, J7 CON3, J8 Conn_01x03_Female, Q1 Q_PNP_BEC, U1 LM358, U2 ISOW7841DWE, U3 THVD1500D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

Commit message: Added missing 5VDC connection to isolator (isow7841dwe) and created new net vcc between isolator and esd/transceiver(thvd1500d). Changed layout.
Parts:
- removed TP5: TestPoint, TestPoint:TestPoint_Loop_D1.80mm_Drill1.0mm_Beaded, symbol Connector:TestPoint
Connections:
- net labels added: vcc
- wire segments 189 -> 188
Changed lines of the file:
@@
 	8675 5050 8675 5150
-Wire Wire Line
-	9000 4950 9375 4950
 Wire Wire Line
 	9000 4050 9000 4950
@@
 Wire Wire Line
 	9425 4650 8675 4650
-$Comp
-L Connector:TestPoint TP5
-U 1 1 5F9E5816
-P 9375 4950
-F 0 "TP5" H 9433 5068 50  0000 L CNN
-F 1 "TestPoint" H 9275 5150 50  0000 L CNN
-F 2 "TestPoint:TestPoint_Loop_D1.80mm_Drill1.0mm_Beaded" H 9575 4950 50  0001 C CNN
-F 3 "~" H 9575 4950 50  0001 C CNN
-	1    9375 4950
-	-1   0    0    1
-$EndComp
-Connection ~ 9375 4950
-Wire Wire Line
-	9375 4950 9500 4950
 Wire Wire Line
 	3500 4600 3600 4600
@@
 	1    0    0    -1
 $EndComp
+Text Label 7425 3100 2    50   ~ 0
+5VDC
+Text Label 8800 3850 0    50   ~ 0
+vcc
+Wire Wire Line
+	9000 4950 9500 4950
 $EndSCHEMATC

Commit message: Headers should now match cc3220modasf commit d3c2dc17dd42c882b5c02795b58cb5e5026f240b
Parts:
- removed J5, J8: Conn_01x03_Female, Connector_PinSocket_2.54mm:PinSocket_1x03_P2.54mm_Vertical, symbol Connector:Conn_01x03_Female
- removed J6: Conn_01x04, Connector_PinSocket_2.54mm:PinSocket_1x04_P2.54mm_Vertical, symbol Connector_Generic:Conn_01x04
- added C12: 0.1u, Capacitor_SMD:C_0603_1608Metric_Pad1.05x0.95mm_HandSolder, symbol Device:C_Small
- added J6, J88: Conn_02x05_Odd_Even, Connector_PinSocket_2.54mm:PinSocket_2x05_P2.54mm_Vertical, symbol Connector_Generic:Conn_02x05_Odd_Even
Connections:
- wire segments 188 -> 187
Changed lines of the file:
@@
 L power:GND #PWR0101
 U 1 1 5D0A6493
-P 3775 6100
-F 0 "#PWR0101" H 3775 5850 50  0001 C CNN
-F 1 "GND" V 3780 5972 50  0000 R CNN
-F 2 "" H 3775 6100 50  0001 C CNN
-F 3 "" H 3775 6100 50  0001 C CNN
-	1    3775 6100
-	0    -1   -1   0
+P 3800 6500
+F 0 "#PWR0101" H 3800 6250 50  0001 C CNN
+F 1 "GND" V 3805 6372 50  0000 R CNN
+F 2 "" H 3800 6500 50  0001 C CNN
+F 3 "" H 3800 6500 50  0001 C CNN
+	1    3800 6500
+	1    0    0    -1
 $EndComp
 $Comp
@@
 $EndComp
 Wire Wire Line
-	3675 7550 3225 7550
+	3675 7550 3600 7550
 Wire Wire Line
 	3225 7550 3225 7350
@@
 Text Notes 7900 1100 0    50   ~ 0
 PowerPax 5V, 1000mA,\n72% efficiency, input current 70mA  \ninrush 20A - 1A/250V slow blow fuse
-Text Label 3675 5750 0    50   ~ 0
+Text Label 3950 6000 0    50   ~ 0
 3V3
 Wire Wire Line
-	3675 6500 3675 6100
-Wire Wire Line
 	3675 6500 3675 7550
-Connection ~ 3675 6500
 Wire Wire Line
 	4350 1550 4750 1550
@@
 $EndComp
 Connection ~ 3225 7050
-$Comp
-L Connector:Conn_01x03_Female J5
-U 1 1 5DA5D055
-P 4150 6400
-F 0 "J5" H 4178 6426 50  0000 L CNN
-F 1 "Conn_01x03_Female" H 4178 6335 50  0000 L CNN
-F 2 "Connector_PinSocket_2.54mm:PinSocket_1x03_P2.54mm_Vertical" H 4150 6400 50  0001 C CNN
-F 3 "~" H 4150 6400 50  0001 C CNN
-	1    4150 6400
-	1    0    0    -1
-$EndComp
 Wire Wire Line
 	3675 6000 3950 6000
 Wire Wire Line
-	3950 6000 3950 6300
-Wire Wire Line
-	3675 6100 3775 6100
-Wire Wire Line
-	3775 6100 3775 6400
-Wire Wire Line
-	3775 6400 3950 6400
-Connection ~ 3775 6100
-Wire Wire Line
-	3775 6400 3775 6500
-Wire Wire Line
-	3775 6500 3950 6500
-Connection ~ 3775 6400
-Wire Wire Line
-	4350 7050 4350 7225
-Wire Wire Line
-	3225 7050 4350 7050
+	3225 7050 3600 7050
 $Comp
 L 2020-09-12_16-45-05:SN74LV1T34DBVR U4
@@
 Wire Wire Line
 	6950 4050 7075 4050
-Text Label 4050 4700 2    50   ~ 0
+Text Label 3500 4500 1    50   ~ 0
 RS485_EN
 Text Label 5375 5925 2    50   ~ 0
@@
 	1075 7550 1825 7550
 Connection ~ 1825 7550
-$Comp
-L Connector:Conn_01x03_Female J8
-U 1 1 5F9513D7
-P 3300 4600
-F 0 "J8" H 3328 4626 50  0000 L CNN
-F 1 "Conn_01x03_Female" H 3328 4535 50  0000 L CNN
-F 2 "Connector_PinSocket_2.54mm:PinSocket_1x03_P2.54mm_Vertical" H 3300 4600 50  0001 C CNN
-F 3 "~" H 3300 4600 50  0001 C CNN
-	1    3300 4600
-	-1   0    0    1
-$EndComp
 Wire Wire Line
 	5450 3775 3600 3775
-Wire Wire Line
-	4050 4700 3500 4700
-Text Label 3500 4500 1    50   ~ 0
+Text Label 3725 5125 2    50   ~ 0
 RS485_RXD
-Text Label 3500 4600 3    50   ~ 0
+Text Label 3600 4600 0    50   ~ 0
 RS485_TXD
 Text Label 1025 7050 1    50   ~ 0
@@
 	3600 4600 3600 3775
 Wire Wire Line
-	3500 4500 3725 4500
-Wire Wire Line
-	3725 4500 3725 5400
-Wire Wire Line
 	8100 1850 8100 2250
 Wire Wire Line
 	6900 2150 6900 2450
-$Comp
-L Connector_Generic:Conn_01x04 J6
-U 1 1 5ECCF259
-P 4250 7425
-F 0 "J6" V 4122 7605 50  0000 L CNN
-F 1 "Conn_01x04" V 4213 7605 50  0000 L CNN
-F 2 "Connector_PinSocket_2.54mm:PinSocket_1x04_P2.54mm_Vertical" H 4250 7425 50  0001 C CNN
-F 3 "~" H 4250 7425 50  0001 C CNN
-	1    4250 7425
-	0    1    1    0
-$EndComp
 $Comp
 L Converter_ACDC:IRM-02-5 PS1
@@
 Wire Wire Line
 	9000 4950 9500 4950
+$Comp
+L Device:C_Small C12
+U 1 1 5F8781FD
+P 3600 7250
+F 0 "C12" H 3692 7296 50  0000 L CNN
+F 1 "0.1u" H 3692 7205 50  0000 L CNN
+F 2 "Capacitor_SMD:C_0603_1608Metric_Pad1.05x0.95mm_HandSolder" H 3600 7250 50  0001 C CNN
+F 3 "~" H 3600 7250 50  0001 C CNN
+F 4 "Kemet" H 3600 7250 50  0001 C CNN "MFG Name"
+F 5 "C0603C104J4RACTU" H 3600 7250 50  0001 C CNN "MFG Part Num"
+	1    3600 7250
+	1    0    0    -1
+$EndComp
+Wire Wire Line
+	3600 7150 3600 7050
+Connection ~ 3600 7050
+Wire Wire Line
+	3600 7350 3600 7550
+Connection ~ 3600 7550
+Wire Wire Line
+	3600 7550 3225 7550
+$Comp
+L Connector_Generic:Conn_02x05_Odd_Even J6
+U 1 1 5FEE70CE
+P 4225 7325
+F 0 "J6" V 4229 7605 50  0000 L CNN
+F 1 "Conn_02x05_Odd_Even" V 4320 7605 50  0000 L CNN
+F 2 "Connector_PinSocket_2.54mm:PinSocket_2x05_P2.54mm_Vertical" H 4225 7325 50  0001 C CNN
+F 3 "~" H 4225 7325 50  0001 C CNN
+	1    4225 7325
+	0    1    1    0
+$EndComp
+Wire Wire Line
+	4425 7125 4425 7050
+Wire Wire Line
+	3600 7050 4425 7050
+$Comp
+L Connector_Generic:Conn_02x05_Odd_Even J88
+U 1 1 5FF2063A
+P 3300 4700
+F 0 "J88" H 3350 4275 50  0000 C CNN
+F 1 "Conn_02x05_Odd_Even" H 3350 4366 50  0000 C CNN
+F 2 "Connector_PinSocket_2.54mm:PinSocket_2x05_P2.54mm_Vertical" H 3300 4700 50  0001 C CNN
+F 3 "~" H 3300 4700 50  0001 C CNN
+	1    3300 4700
+	-1   0    0    1
+$EndComp
+$Comp
+L power:GND #PWR0115
+U 1 1 5F84025E
+P 3000 4900
+F 0 "#PWR0115" H 3000 4650 50  0001 C CNN
+F 1 "GND" H 3005 4727 50  0000 C CNN
+F 2 "" H 3000 4900 50  0001 C CNN
+F 3 "" H 3000 4900 50  0001 C CNN
+	1    3000 4900
+	1    0    0    -1
+$EndComp
+Text Label 3500 4900 0    50   ~ 0
+3V3
+Wire Wire Line
+	3500 4700 3725 4700
+Wire Wire Line
+	3725 4700 3725 5400
+Wire Wire Line
+	3500 4500 4050 4500
+Wire Wire Line
+	4050 4500 4050 4700
+Wire Wire Line
+	3675 6500 3800 6500
+Connection ~ 3675 6500
 $EndSCHEMATC

Commit message: State at time of 2021-11-25 Aisler order
Parts:
- removed D1: D, Diode_SMD:D_SOD-123, symbol Device:D
- added R13: 0, Resistor_SMD:R_0603_1608Metric, symbol Device:R
- added TP1, TP3: TestPoint, TestPoint:TestPoint_THTPad_D1.5mm_Drill0.7mm, symbol Connector:TestPoint
- C10: value 1u -> 4u7; MFG Name (none) -> AVX; MFG Part Num (none) -> F981A475MMA
- C11: MFG Name (none) -> Murata; MFG Part Num (none) -> ‎GRM033R61E471KA01D‎
- TP2: renamed from TP4; footprint TestPoint:TestPoint_Loop_D1.80mm_Drill1.0mm_Beaded -> TestPoint:TestPoint_Pad_D1.5mm
- U1: value LM358 -> LM358M; footprint Package_DIP:DIP-8_W7.62mm -> Package_SO:SOIC-8-1EP_3.9x4.9mm_P1.27mm_EP2.29x3mm; MFG Name (none) -> Texas Instruments; MFG Part Num (none) -> LM358M/NOPB
Connections:
- net Q1E is gone; now on net 3V3: Q1.2 (E), R1.1
- net 3V3: now also R13.2; no longer C10.1, U7.3 (OUT)
- net 5VDC: now also J88.9 (Pin_9)
- net GND: now also J88.10 (Pin_10), J88.8 (Pin_8)
- net RS485_EN: now also J88.7 (Pin_7); no longer J88.9 (Pin_9)
- net RS485_RXD: now also J88.3 (Pin_3); no longer J88.5 (Pin_5)
- net RS485_TXD: now also J88.5 (Pin_5); no longer J88.7 (Pin_7)
- net at U2.11 (IND), U3.1 (R): now also TP3.1; no longer TP2.1
- net at U2.12 (OUTC), U3.3 (DE): now also TP1.1
- net at U2.14 (OUTA), U3.4 (D): now also TP2.1
- new net: C10.1, R13.1, U7.3 (OUT)
Other:
- moved on the sheet: TP2
Changed lines of the file:
@@
-	1    0    0    -1
-$EndComp
-$Comp
-L Device:D D1
-U 1 1 5D0A80F4
-P 2475 5750
-F 0 "D1" H 2475 5966 50  0000 C CNN
-F 1 "D" H 2475 5875 50  0000 C CNN
-F 2 "Diode_SMD:D_SOD-123" H 2475 5750 50  0001 C CNN
-F 3 "~" H 2475 5750 50  0001 C CNN
-F 4 "Diodes Inc" H 2475 5750 50  0001 C CNN "MFG Name"
-F 5 " BAV16W-7-F" H 2475 5750 50  0001 C CNN "MFG Part Num"
-	1    2475 5750
 	1    0    0    -1
 $EndComp
@@
 P 2575 7050
 F 0 "U1" H 2575 7417 50  0000 C CNN
-F 1 "LM358" H 2575 7326 50  0000 C CNN
-F 2 "Package_DIP:DIP-8_W7.62mm" H 2575 7050 50  0001 C CNN
-F 3 "http://www.ti.com/lit/ds/symlink/lm2904-n.pdf" H 2575 7050 50  0001 C CNN
+F 1 "LM358M" H 2575 7326 50  0000 C CNN
+F 2 "Package_SO:SOIC-8-1EP_3.9x4.9mm_P1.27mm_EP2.29x3mm" H 2575 7050 50  0001 C CNN
+F 3 "~/dev/kicad/mov/pwrcon_1/docs/lm358-n.pdf" H 2575 7050 50  0001 C CNN
+F 4 "Texas Instruments" H 2575 7050 50  0001 C CNN "MFG Name"
+F 5 "LM358M/NOPB" H 2575 7050 50  0001 C CNN "MFG Part Num"
 	2    2575 7050
 	1    0    0    -1
@@
 Wire Wire Line
 	3225 7550 3225 7350
-Wire Wire Line
-	2625 5750 3675 5750
 $Comp
 L Device:R_Small R5
@@
 Text Notes 7900 1100 0    50   ~ 0
 PowerPax 5V, 1000mA,\n72% efficiency, input current 70mA  \ninrush 20A - 1A/250V slow blow fuse
-Text Label 3950 6000 0    50   ~ 0
+Text Label 2325 5750 0    50   ~ 0
 3V3
 Wire Wire Line
@@
 P 2575 7050
 F 0 "U1" H 2533 7096 50  0000 L CNN
-F 1 "LM358" H 2533 7005 50  0000 L CNN
-F 2 "Package_DIP:DIP-8_W7.62mm" H 2575 7050 50  0001 C CNN
-F 3 "http://www.ti.com/lit/ds/symlink/lm2904-n.pdf" H 2575 7050 50  0001 C CNN
+F 1 "LM358M" H 2533 7005 50  0000 L CNN
+F 2 "Package_SO:SOIC-8-1EP_3.9x4.9mm_P1.27mm_EP2.29x3mm" H 2575 7050 50  0001 C CNN
+F 3 "~/dev/kicad/mov/pwrcon_1/lm358-n.pdf" H 2575 7050 50  0001 C CNN
+F 4 "Texas Instruments" H 2575 7050 50  0001 C CNN "MFG Name"
+F 5 "LM358M/NOPB" H 2575 7050 50  0001 C CNN "MFG Part Num"
 	3    2575 7050
 	1    0    0    -1
@@
 $EndComp
 Wire Wire Line
-	3675 6000 3675 5750
-Wire Wire Line
 	1125 7050 1125 7150
 Wire Wire Line
@@
 Connection ~ 3225 7050
 Wire Wire Line
-	3675 6000 3950 6000
-Wire Wire Line
 	3225 7050 3600 7050
 $Comp
@@
 Text Notes 9950 3600 0    50   ~ 0
 Isolated RS485 Transceiver
-Wire Wire Line
-	7075 4250 7075 4450
 Connection ~ 8675 5150
 $Comp
@@
 	9200 4750 9500 4750
 Wire Wire Line
-	9200 4250 9200 4750
-Wire Wire Line
 	8675 4250 9200 4250
-Wire Wire Line
-	9500 4650 9425 4650
 $Comp
 L 2020-09-12_17-09-47:ISOW7841DWE U2
@@
 Wire Wire Line
 	6950 4050 7075 4050
-Text Label 3500 4500 1    50   ~ 0
+Text Label 4050 4600 2    50   ~ 0
 RS485_EN
 Text Label 5375 5925 2    50   ~ 0
@@
 Wire Wire Line
 	5550 4700 6725 4700
-Connection ~ 7075 4450
-$Comp
-L Connector:TestPoint TP4
+$Comp
+L Connector:TestPoint TP2
 U 1 1 5F74616A
-P 9425 4650
-F 0 "TP4" H 9483 4768 50  0000 L CNN
-F 1 "TestPoint" H 9325 4850 50  0000 L CNN
-F 2 "TestPoint:TestPoint_Loop_D1.80mm_Drill1.0mm_Beaded" H 9625 4650 50  0001 C CNN
-F 3 "~" H 9625 4650 50  0001 C CNN
-	1    9425 4650
-	1    0    0    -1
+P 9000 4050
+F 0 "TP2" H 9058 4168 50  0000 L CNN
+F 1 "TestPoint" H 8900 4250 50  0000 L CNN
+F 2 "TestPoint:TestPoint_Pad_D1.5mm" H 9200 4050 50  0001 C CNN
+F 3 "~" H 9200 4050 50  0001 C CNN
+	1    9000 4050
+	0    1    1    0
 $EndComp
 $Comp
@@
 Text Label 3725 5125 2    50   ~ 0
 RS485_RXD
-Text Label 3600 4600 0    50   ~ 0
+Text Label 3600 4700 0    50   ~ 0
 RS485_TXD
 Text Label 1025 7050 1    50   ~ 0
@@
 	1    0    0    -1
 $EndComp
-Text Label 2150 3700 0    50   ~ 0
+Text Label 2625 3700 1    50   ~ 0
 3V3
 Text Label 1550 3700 2    50   ~ 0
@@
 U 1 1 5F769B74
 P 2325 3800
-F 0 "C10" H 2417 3846 50  0000 L CNN
-F 1 "1u" H 2417 3755 50  0000 L CNN
+F 0 "C10" H 2400 3800 50  0000 L CNN
+F 1 "4u7" H 2400 3725 50  0000 L CNN
 F 2 "Capacitor_SMD:C_0603_1608Metric_Pad1.05x0.95mm_HandSolder" H 2325 3800 50  0001 C CNN
 F 3 "~" H 2325 3800 50  0001 C CNN
+F 4 "AVX" H 2325 3800 50  0001 C CNN "MFG Name"
+F 5 "F981A475MMA" H 2325 3800 50  0001 C CNN "MFG Part Num"
 	1    2325 3800
 	1    0    0    -1
@@
 U 1 1 5F791E36
 P 2150 3900
-F 0 "C11" H 2242 3946 50  0000 L CNN
-F 1 "470p" H 2242 3855 50  0000 L CNN
+F 0 "C11" H 2225 3875 50  0000 L CNN
+F 1 "470p" H 2150 3800 50  0000 L CNN
 F 2 "Capacitor_SMD:C_0603_1608Metric_Pad1.05x0.95mm_HandSolder" H 2150 3900 50  0001 C CNN
 F 3 "~" H 2150 3900 50  0001 C CNN
+F 4 "Murata" H 2150 3900 50  0001 C CNN "MFG Name"
+F 5 "‎GRM033R61E471KA01D‎" H 2150 3900 50  0001 C CNN "MFG Part Num"
 	1    2150 3900
 	1    0    0    -1
@@
 Wire Wire Line
 	4950 5925 5375 5925
-Connection ~ 9425 4650
-Wire Wire Line
-	9425 4650 8675 4650
-Wire Wire Line
-	3500 4600 3600 4600
-Wire Wire Line
-	3600 4600 3600 3775
 Wire Wire Line
 	8100 1850 8100 2250
@@
 3V3
 Wire Wire Line
-	3500 4700 3725 4700
-Wire Wire Line
-	3725 4700 3725 5400
-Wire Wire Line
-	3500 4500 4050 4500
-Wire Wire Line
-	4050 4500 4050 4700
-Wire Wire Line
 	3675 6500 3800 6500
 Connection ~ 3675 6500
+Wire Wire Line
+	3500 4800 3725 4800
+Wire Wire Line
+	3725 4800 3725 5400
+Wire Wire Line
+	3500 4700 3600 4700
+Wire Wire Line
+	4050 4600 4050 4700
+Wire Wire Line
+	3600 3775 3600 4700
+Wire Wire Line
+	3500 4600 4050 4600
+Wire Wire Line
+	7075 4250 7075 4450
+Connection ~ 7075 4450
+Text Label 3500 4500 0    50   ~ 0
+5VDC
+$Comp
+L power:GND #PWR0116
+U 1 1 5FBCB498
+P 3000 4500
+F 0 "#PWR0116" H 3000 4250 50  0001 C CNN
+F 1 "GND" V 3005 4372 50  0000 R CNN
+F 2 "" H 3000 4500 50  0001 C CNN
+F 3 "" H 3000 4500 50  0001 C CNN
+	1    3000 4500
+	0    1    1    0
+$EndComp
+$Comp
+L power:GND #PWR0117
+U 1 1 5FC26E34
+P 3000 4600
+F 0 "#PWR0117" H 3000 4350 50  0001 C CNN
+F 1 "GND" V 3005 4472 50  0000 R CNN
+F 2 "" H 3000 4600 50  0001 C CNN
+F 3 "" H 3000 4600 50  0001 C CNN
+	1    3000 4600
+	0    1    1    0
+$EndComp
+$Comp
+L Device:R R13
+U 1 1 5FC6C320
+P 2475 3700
+F 0 "R13" V 2550 3825 50  0000 C CNN
+F 1 "0" V 2575 3700 50  0000 C CNN
+F 2 "Resistor_SMD:R_0603_1608Metric" V 2405 3700 50  0001 C CNN
+F 3 "~" H 2475 3700 50  0001 C CNN
+F 4 "Y" V 2475 3700 50  0001 C CNN "Fit"
+F 5 "Rohm" H 2475 3700 50  0001 C CNN "MFG Name"
+F 6 "ESR03EZPJ152" H 2475 3700 50  0001 C CNN "MFG Part Num"
+	1    2475 3700
+	0    -1   -1   0
+$EndComp
+Connection ~ 2325 3700
+Connection ~ 9000 4050
+Wire Wire Line
+	8675 4650 8850 4650
+$Comp
+L Connector:TestPoint TP1
+U 1 1 5FCB900E
+P 9075 4450
+F 0 "TP1" H 9133 4568 50  0000 L CNN
+F 1 "TestPoint" H 8975 4650 50  0000 L CNN
+F 2 "TestPoint:TestPoint_THTPad_D1.5mm_Drill0.7mm" H 9275 4450 50  0001 C CNN
+F 3 "~" H 9275 4450 50  0001 C CNN
+	1    9075 4450
+	0    1    1    0
+$EndComp
+$Comp
+L Connector:TestPoint TP3
+U 1 1 5FCC1982
+P 8850 4650
+F 0 "TP3" H 8908 4768 50  0000 L CNN
+F 1 "TestPoint" H 8750 4850 50  0000 L CNN
+F 2 "TestPoint:TestPoint_THTPad_D1.5mm_Drill0.7mm" H 9050 4650 50  0001 C CNN
+F 3 "~" H 9050 4650 50  0001 C CNN
+	1    8850 4650
+	-1   0    0    1
+$EndComp
+Connection ~ 8850 4650
+Wire Wire Line
+	8850 4650 9500 4650
+Connection ~ 9075 4450
+Wire Wire Line
+	9200 4250 9200 4750
 $EndSCHEMATC
